File: icncconv.kicad_sch (KiCad schematic)
At the start: 31 parts, among them J1 Conn_01x11_Pin, J3 Conn_01x11_Pin, SW1 SW_SPDT, U1 iC-NV, U2 MC3487N

Commit message: up EMI
Parts:
- removed H4: MountingHole, MountingHole:MountingHole_3.2mm_M3, symbol Mechanical:MountingHole
- removed SW1: SW_SPDT, easyeda2kicad:SW-SMD_CJS-1201B, symbol Switch:SW_SPDT
- added C10, C11, C12, C13, C14, C15, C16, C8, C9: 470p, Capacitor_SMD:C_1206_3216Metric_Pad1.33x1.80mm_HandSolder, symbol Device:C
- added C17: 4n7, Capacitor_SMD:C_1206_3216Metric_Pad1.33x1.80mm_HandSolder, symbol Device:C
- added D1, D10, D11, D12, D2, D3, D4, D5, D6, D7, D8, D9: SD15_SOD323, Diode_SMD:D_SOD-323, symbol Diode:SD15_SOD323
- added H5: MountingHole_Pad, MountingHole:MountingHole_3.2mm_M3_Pad, symbol Mechanical:MountingHole_Pad
- added R1, R11, R12, R13, R2: 1K, Resistor_SMD:R_1206_3216Metric_Pad1.30x1.75mm_HandSolder, symbol Device:R
- added R3, R4: 25K, Resistor_SMD:R_1206_3216Metric_Pad1.30x1.75mm_HandSolder, symbol Device:R
- added SW1: SS-3292S-L2-B, easyeda2kicad:SW-SMD_SS-3292S-L2-B, symbol easyeda2kicad:SS-3292S-L2-B
- R10: value 25K -> 1M
- R5: value 25K -> 1K
Connections:
- net +5V: now also SW1.1
- net A+: now also U2.6 (2Y), D7.2 (A2); no longer U2.2 (1Y)
- net A-: now also U2.5 (2Z), D8.2 (A2); no longer U2.3 (1Z)
- net B+: now also U2.2 (1Y), D9.2 (A2); no longer U2.6 (2Y)
- net B-: now also U2.3 (1Z), D10.2 (A2); no longer U2.5 (2Z)
- net COS+: now also C11.1, C12.1, D2.2 (A2), R2.1, R2.2, R3.2; no longer R7.2
- net COS-: now also C12.2, C13.2, D1.1 (A1), R13.1, R13.2, R4.1; no longer R10.1
- net GND: now also R10.2, C10.1, C11.2, C13.1, C14.2, C16.1, C17.2, C8.2, D1.2 (A2), D10.1 (A1), D11.1 (A1), D12.1 (A1), D2.1 (A1), D3.2 (A2), D4.1 (A1), D5.2 (A2), D6.1 (A1), D7.1 (A1), D8.1 (A1), D9.1 (A1), SW1.EH
- net ICNV_RCLK: now also SW1.2
- net ICNV_VREF: now also R7.2, R9.2, R3.1, R4.2; no longer R10.2, R5.1, R7.1, R9.1
- net IDX+: now also R5.1, R6.2, C14.1, C15.1, D4.2 (A2)
- net IDX-: now also R7.1, C15.2, C16.2, D3.1 (A1), R12.1, R12.2; no longer R6.2
- net MC_1A: now also U2.7 (2A); no longer U2.1 (1A)
- net MC_2A: now also U2.1 (1A); no longer U2.7 (2A)
- net MC_3A: now also U2.15 (4A); no longer U2.9 (3A)
- net SHIELD: no longer J1.10 (Pin_10), J1.11 (Pin_11), J3.10 (Pin_10), J3.11 (Pin_11)
- net SIN+: now also C8.1, C9.1, D6.2 (A2), R1.1, R1.2
- net SIN-: now also R9.1, C10.2, C9.2, D5.1 (A1), R11.1, R11.2; no longer R9.2
- net Z+: now also U2.14 (4Y), D11.2 (A2); no longer U2.10 (3Y)
- net Z-: now also U2.13 (4Z), D12.2 (A2); no longer U2.11 (3Z)
- net at RV3.2, RV3.3, TP1.1: now also SW1.3
- new net GNDS: C17.1, H5.1, J1.10 (Pin_10), J1.11 (Pin_11), J3.10 (Pin_10), J3.11 (Pin_11), R10.1
Other:
- moved on the sheet: R8, R9

Commit message: update
Parts:
- added D13: LED, easyeda2kicad:LED-SMD_L3.2-W1.0-R-RD_GREEN, symbol Device:LED
- added R14: 150, Resistor_SMD:R_0603_1608Metric_Pad0.98x0.95mm_HandSolder, symbol Device:R
- C1, C10, C11, C12, C13, C14, C15, C16, C17, C2, C3, C4, C5, C6, C7, C8, C9: footprint Capacitor_SMD:C_1206_3216Metric_Pad1.33x1.80mm_HandSolder -> Capacitor_SMD:C_0603_1608Metric_Pad1.08x0.95mm_HandSolder
- R1, R10, R11, R12, R13, R2, R3, R4, R5, R6, R7, R8, R9: footprint Resistor_SMD:R_1206_3216Metric_Pad1.30x1.75mm_HandSolder -> Resistor_SMD:R_0603_1608Metric_Pad0.98x0.95mm_HandSolder
Connections:
- net +5V: now also D13.2 (A)
- net GND: now also R14.2
- new net: D13.1 (K), R14.1
