File: icncconv.kicad_pcb (KiCad board)
At the start: 4 copper layers, 70.3 x 50 mm, 31 parts, among them J1 Conn_01x11_Pin, J3 Conn_01x11_Pin, SW1 SW_SPDT, U1 iC-NV, U2 MC3487N

Commit message: up EMI
Parts:
- removed H4: MountingHole, MountingHole:MountingHole_3.2mm_M3
- added C10: 470p, Capacitor_SMD:C_1206_3216Metric_Pad1.33x1.80mm_HandSolder, F.Cu at (138.7, 99.8)
- added C11: 470p, Capacitor_SMD:C_1206_3216Metric_Pad1.33x1.80mm_HandSolder, F.Cu at (141.6, 102.3)
- added C12: 470p, Capacitor_SMD:C_1206_3216Metric_Pad1.33x1.80mm_HandSolder, F.Cu at (138.7, 105.4)
- added C13: 470p, Capacitor_SMD:C_1206_3216Metric_Pad1.33x1.80mm_HandSolder, F.Cu at (141.6, 108.5)
- added C14: 470p, Capacitor_SMD:C_1206_3216Metric_Pad1.33x1.80mm_HandSolder, F.Cu at (141.7, 85.5)
- added C15: 470p, Capacitor_SMD:C_1206_3216Metric_Pad1.33x1.80mm_HandSolder, F.Cu at (138.7, 88.6)
- added C16: 470p, Capacitor_SMD:C_1206_3216Metric_Pad1.33x1.80mm_HandSolder, F.Cu at (141.7, 91.7)
- added C17: 4n7, Capacitor_SMD:C_1206_3216Metric_Pad1.33x1.80mm_HandSolder, F.Cu at (168.8, 119.8)
- added C8: 470p, Capacitor_SMD:C_1206_3216Metric_Pad1.33x1.80mm_HandSolder, F.Cu at (138.7, 94.3)
- added C9: 470p, Capacitor_SMD:C_1206_3216Metric_Pad1.33x1.80mm_HandSolder, F.Cu at (141.6, 97.0)
- added D1: SD15_SOD323, Diode_SMD:D_SOD-323, F.Cu at (123.5, 107.4)
- added D10: SD15_SOD323, Diode_SMD:D_SOD-323, F.Cu at (175.8, 99.3)
- added D11: SD15_SOD323, Diode_SMD:D_SOD-323, F.Cu at (175.8, 104.5)
- added D12: SD15_SOD323, Diode_SMD:D_SOD-323, F.Cu at (175.8, 107.3)
- added D2: SD15_SOD323, Diode_SMD:D_SOD-323, F.Cu at (123.5, 103.3)
- added D3: SD15_SOD323, Diode_SMD:D_SOD-323, F.Cu at (123.5, 90.7)
- added D4: SD15_SOD323, Diode_SMD:D_SOD-323, F.Cu at (123.5, 86.6)
- added D5: SD15_SOD323, Diode_SMD:D_SOD-323, F.Cu at (123.5, 98.9)
- added D6: SD15_SOD323, Diode_SMD:D_SOD-323, F.Cu at (123.5, 95.2)
- added D7: SD15_SOD323, Diode_SMD:D_SOD-323, F.Cu at (175.8, 93.6)
- added D8: SD15_SOD323, Diode_SMD:D_SOD-323, F.Cu at (175.8, 96.3)
- added D9: SD15_SOD323, Diode_SMD:D_SOD-323, F.Cu at (175.8, 102.1)
- added H5: MountingHole_Pad, MountingHole:MountingHole_3.2mm_M3_Pad, F.Cu at (176.5, 119.8)
- added R1: 1K, Resistor_SMD:R_1206_3216Metric_Pad1.30x1.75mm_HandSolder, F.Cu at (133.9, 95.7)
- added R11: 1K, Resistor_SMD:R_1206_3216Metric_Pad1.30x1.75mm_HandSolder, F.Cu at (133.9, 98.4)
- added R12: 1K, Resistor_SMD:R_1206_3216Metric_Pad1.30x1.75mm_HandSolder, F.Cu at (133.9, 90.2)
- added R13: 1K, Resistor_SMD:R_1206_3216Metric_Pad1.30x1.75mm_HandSolder, F.Cu at (133.9, 107.0)
- added R2: 1K, Resistor_SMD:R_1206_3216Metric_Pad1.30x1.75mm_HandSolder, F.Cu at (133.9, 103.8)
- added R3: 25K, Resistor_SMD:R_1206_3216Metric_Pad1.30x1.75mm_HandSolder, F.Cu at (128.1, 103.8)
- added R4: 25K, Resistor_SMD:R_1206_3216Metric_Pad1.30x1.75mm_HandSolder, F.Cu at (128.1, 107.0)
- R10: value 25K -> 1M
- R5: value 25K -> 1K
- SW1: value SW_SPDT -> SS-3292S-L2-B; footprint easyeda2kicad:SW-SMD_CJS-1201B -> easyeda2kicad:SW-SMD_SS-3292S-L2-B
- moved R10 34.9 mm to (168.8, 115.6), turned to 180 degrees
- moved R7 13.0 mm to (128.1, 90.2), turned to 0 degrees
- moved H1 12.5 mm to (120.8, 80.8)
- moved H3 12.5 mm to (120.8, 119.9)
- moved C2 9.54 mm to (123.5, 112.4)
- moved R6 9.50 mm to (128.1, 87.1)
- moved J1 9.29 mm to (117.6, 100.5)
- moved R8 8.06 mm to (128.1, 95.7)
- moved R9 8.06 mm to (128.1, 98.4), turned to 0 degrees
- moved H2 4.19 mm to (176.5, 80.7)
- moved C1 3.34 mm to (151.1, 112.0)
- moved JP1 3.34 mm to (145.1, 111.9)
- moved JP2 3.34 mm to (148.3, 111.9)
- moved JP3 3.34 mm to (157.2, 111.9)
- moved JP4 3.34 mm to (154.0, 111.9)
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Connections:
- J1 pad 10: SHIELD -> GNDS
- J1 pad 11: SHIELD -> GNDS
- J3 pad 10: SHIELD -> GNDS
- J3 pad 11: SHIELD -> GNDS
- R10 pad 1: COS- -> GNDS
- R10 pad 2: ICNV_VREF -> GND
- R5 pad 1: ICNV_VREF -> IDX+
- R6 pad 2: IDX- -> IDX+
- R7 pad 1: ICNV_VREF -> IDX-
- R7 pad 2: COS+ -> ICNV_VREF
- R9 pad 1: ICNV_VREF -> SIN-
- R9 pad 2: SIN- -> ICNV_VREF
- U2 pad 1: MC_1A -> MC_2A
- U2 pad 10: Z+ -> unconnected-(U2-3Y-Pad10)
- U2 pad 11: Z- -> unconnected-(U2-3Z-Pad11)
- U2 pad 13: unconnected-(U2-4Z-Pad13) -> Z-
- U2 pad 14: unconnected-(U2-4Y-Pad14) -> Z+
- U2 pad 15: unconnected-(U2-4A-Pad15) -> MC_3A
- U2 pad 2: A+ -> B+
- U2 pad 3: A- -> B-
- U2 pad 5: B- -> A-
- U2 pad 6: B+ -> A+
- U2 pad 7: MC_2A -> MC_1A
- U2 pad 9: MC_3A -> unconnected-(U2-3A-Pad9)
Routing:
- net GNDS: track 0.00 -> 142.0 mm
- net GND: track 23.8 -> 81.5 mm, vias 15 -> 65
- net SHIELD: track 121.6 -> 95.1 mm
- net IDX+: track 34.7 -> 48.9 mm
- net IDX-: track 34.8 -> 49.0 mm
- net A+: track 7.45 -> 18.9 mm
- net SIN-: track 23.8 -> 34.9 mm
- net SIN+: track 23.8 -> 34.9 mm
- net COS-: track 26.0 -> 36.9 mm
- net COS+: track 26.0 -> 36.8 mm
- net A-: track 8.31 -> 17.5 mm
- net MC_1A: track 21.9 -> 12.8 mm
- net MC_3A: track 9.16 -> 17.8 mm
- net +5V: track 43.0 -> 51.4 mm
- net ICNV_VREF: track 73.9 -> 81.6 mm, vias 6 -> 8
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Other:
- board size 70.3 x 50 mm -> 82.9 x 50 mm

Commit message: up
Routing:
- net B+: track 12.8 -> 15.8 mm
- net A-: track 17.5 -> 18.8 mm
- net Z-: track 15.0 -> 15.6 mm

Commit message: update
Parts:
- added D13: LED, easyeda2kicad:LED-SMD_L3.2-W1.0-R-RD_GREEN, F.Cu at (136.7, 116.3)
- added R14: 150, Resistor_SMD:R_0603_1608Metric_Pad0.98x0.95mm_HandSolder, F.Cu at (142.4, 116.1)
- C1, C10, C11, C12, C13, C14, C15, C16, C17, C2, C3, C4, C5, C6, C7, C8, C9: footprint Capacitor_SMD:C_1206_3216Metric_Pad1.33x1.80mm_HandSolder -> Capacitor_SMD:C_0603_1608Metric_Pad1.08x0.95mm_HandSolder
- R1, R10, R11, R12, R13, R2, R3, R4, R5, R6, R7, R8, R9: footprint Resistor_SMD:R_1206_3216Metric_Pad1.30x1.75mm_HandSolder -> Resistor_SMD:R_0603_1608Metric_Pad0.98x0.95mm_HandSolder
- moved D1 6.53 mm to (130.0, 107.0)
- moved C2 6.53 mm to (130.0, 112.4)
- moved D2 6.53 mm to (130.0, 103.3)
- moved D3 6.53 mm to (130.0, 90.6)
- moved D5 6.53 mm to (130.0, 98.9)
- moved D6 6.53 mm to (130.0, 95.2)
- moved H1 6.53 mm to (127.4, 80.8)
- moved H3 6.53 mm to (127.4, 119.9)
- moved J1 6.53 mm to (124.1, 100.4)
- moved D4 6.53 mm to (130.0, 86.9)
- moved R4 4.95 mm to (133.0, 106.2)
- moved R6 4.94 mm to (133.0, 87.8)
- moved R7 4.91 mm to (133.0, 89.8)
- moved R9 4.90 mm to (133.0, 98.0)
- moved R3 4.90 mm to (133.0, 104.2)
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Routing:
- net IDX-: track 49.0 -> 40.8 mm
- net IDX+: track 48.9 -> 40.7 mm
- net COS-: track 36.9 -> 29.2 mm
- net COS+: track 36.8 -> 29.2 mm
- net SIN+: track 34.9 -> 28.3 mm
- net SIN-: track 34.9 -> 28.3 mm
- net SHIELD: track 95.1 -> 88.5 mm
- net GNDS: track 142.0 -> 138.0 mm
- net ICNV_VREF: track 81.6 -> 85.5 mm, vias 8 -> 6
- net Net-(D13-K): track 0.00 -> 3.49 mm
- net GNDA: track 9.48 -> 7.37 mm
- net +5V: track 51.4 -> 52.2 mm, vias 7 -> 8
- net GND: track 81.5 -> 80.7 mm
Other:
- board size 82.9 x 50 mm -> 76.4 x 50.1 mm
- board text removed: "R6"

Commit message: update prodv1
Routing:
- net SHIELD: track 88.5 -> 108.5 mm
Other:
- board text removed: "25K"
